Commit message: refactor: robot1_description to robot_description

File: ws_ros1/src/robot_description/urdf/robot1.urdf (robot description, URDF)
Before this commit: robot origins, 12 links, 11 joints
Links:
- link left_gripper: geometry collision box size=0.1 .1 .1; visual mesh filename=package://robot_description/meshes/gripper_v0/l_finger.dae
- link left_tip: geometry collision box size=0.1 .1 .1; visual mesh filename=package://robot_description/meshes/gripper_v0/l_finger_tip.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
- link right_gripper: geometry collision box size=0.1 .1 .1; visual mesh filename=package://robot_description/meshes/gripper_v0/l_finger.dae
- link right_tip: geometry collision box size=0.1 .1 .1; visual mesh filename=package://robot_description/meshes/gripper_v0/l_finger_tip.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

File: ws_ros1/src/robot_description/urdf/robot1.xacro (robot description, xacro)
@@ -204,5 +204,5 @@
 			<origin rpy="0 0 0" xyz="0 0 0"/>
 			<geometry>
-				<mesh filename="package://robot1_description/meshes/gripper_v0/l_finger.dae"/>
+				<mesh filename="package://robot_description/meshes/gripper_v0/l_finger.dae"/>
 			</geometry>
 		</visual>
@@ -222,5 +222,5 @@
 			<origin rpy="0.0 0 0" xyz="0.09137 0.00495 0"/>
 			<geometry>
-				<mesh filename="package://robot1_description/meshes/gripper_v0/l_finger_tip.dae"/>
+				<mesh filename="package://robot_description/meshes/gripper_v0/l_finger_tip.dae"/>
 			</geometry>
 		</visual>
@@ -243,5 +243,5 @@
 			<origin rpy="-3.1415 0 0" xyz="0 0 0"/>
 			<geometry>
-				<mesh filename="package://robot1_description/meshes/gripper_v0/l_finger.dae"/>
+				<mesh filename="package://robot_description/meshes/gripper_v0/l_finger.dae"/>
 			</geometry>
 		</visual>
@@ -261,5 +261,5 @@
 			<origin rpy="-3.1415 0 0" xyz="0.09137 0.00495 0"/>
 			<geometry>
-				<mesh filename="package://robot1_description/meshes/gripper_v0/l_finger_tip.dae"/>
+				<mesh filename="package://robot_description/meshes/gripper_v0/l_finger_tip.dae"/>
 			</geometry>
 		</visual>

File: ws_ros1/src/robot_description/urdf/robot1_arm.xacro (robot description, xacro)
@@ -86,5 +86,5 @@
 			<origin rpy="0 0 0" xyz="0 0 0"/>
 			<geometry>
-				<mesh filename="package://robot1_description/meshes/gripper_v0/l_finger.dae"/>
+				<mesh filename="package://robot_description/meshes/gripper_v0/l_finger.dae"/>
 			</geometry>
 		</visual>
@@ -104,5 +104,5 @@
 			<origin rpy="0.0 0 0" xyz="0.09137 0.00495 0"/>
 			<geometry>
-				<mesh filename="package://robot1_description/meshes/gripper_v0/l_finger_tip.dae"/>
+				<mesh filename="package://robot_description/meshes/gripper_v0/l_finger_tip.dae"/>
 			</geometry>
 		</visual>
@@ -125,5 +125,5 @@
 			<origin rpy="-3.1415 0 0" xyz="0 0 0"/>
 			<geometry>
-				<mesh filename="package://robot1_description/meshes/gripper_v0/l_finger.dae"/>
+				<mesh filename="package://robot_description/meshes/gripper_v0/l_finger.dae"/>
 			</geometry>
 		</visual>
@@ -143,5 +143,5 @@
 			<origin rpy="-3.1415 0 0" xyz="0.09137 0.00495 0"/>
 			<geometry>
-				<mesh filename="package://robot1_description/meshes/gripper_v0/l_finger_tip.dae"/>
+				<mesh filename="package://robot_description/meshes/gripper_v0/l_finger_tip.dae"/>
 			</geometry>
 		</visual>

File: ws_ros1/src/robot_description/urdf/robot1_base_01_cam.xacro (robot description, xacro)
@@ -22,5 +22,5 @@
 		<xacro:default_inertial mass="0.0001"/>
 	</link>
-	<xacro:include filename="$(find robot1_description)/urdf/robot.gazebo" />
+	<xacro:include filename="$(find robot_description)/urdf/robot.gazebo" />
 	<gazebo reference="base_footprint">
 		<material>Gazebo/Green</material>
@@ -118,5 +118,5 @@
 		<parent link="base_link"/>
 		<child link="wheel_1"/>
-		<origin rpy="-1.5707 0 0" xyz="0.1 0.15 0"/>
+		<origin rpy="1.5707 0 0" xyz="0.1 0.15 0"/>
 		<axis xyz="0 0 1" />
 	</joint>
@@ -127,5 +127,5 @@
 		<parent link="base_link"/>
 		<child link="wheel_2"/>
-		<origin rpy="-1.5707 0 0" xyz="-0.1 0.15 0"/>
+		<origin rpy="1.5707 0 0" xyz="-0.1 0.15 0"/>
 	</joint>
 	<joint name="base_to_wheel3" type="continuous">
@@ -133,5 +133,5 @@
 		<axis xyz="0 0 1" />
 		<child link="wheel_3"/>
-		<origin rpy="-1.5707 0 0" xyz="0.1 -0.15 0"/>
+		<origin rpy="1.5707 0 0" xyz="0.1 -0.15 0"/>
 	</joint>
 	<joint name="base_to_wheel4" type="continuous">
@@ -139,7 +139,6 @@
 		<axis xyz="0 0 1" />
 		<child link="wheel_4"/>
-		<origin rpy="-1.5707 0 0" xyz="-0.1 -0.15 0"/>
+		<origin rpy="1.5707 0 0" xyz="-0.1 -0.15 0"/>
 	</joint>
-	<!-- Camera joint -->
 	<joint name="camera_joint" type="fixed">
 		<axis xyz="0 1 0" />
@@ -171,47 +170,3 @@
 		</inertial>
 	</link>
-	<!-- Hokuyo joint -->
-	<joint name="hokuyo_joint" type="fixed">
-		<origin xyz="0.125 0.05 0.125" rpy="0 0 0"/>
-		<parent link="base_link"/>
-		<axis xyz="0 1 0" />
-		<child link="hokuyo_link"/>
-	</joint>
-	<!-- Hokuyo Laser -->
-	<link name="hokuyo_link">
-		<collision>
-			<origin xyz="0 0 0" rpy="0 0 0"/>
-			<geometry>
-				<box size="0.1 0.1 0.1"/>
-			</geometry>
-		</collision>
-		<visual>
-			<origin xyz="0 0 0" rpy="0 0 0"/>
-			<geometry>
-				<mesh filename="package://robot1_description/meshes/hokuyo.dae"/>
-			</geometry>
-		</visual>
-		<inertial>
-			<mass value="1e-5" />
-			<origin xyz="0 0 0" rpy="0 0 0"/>
-			<inertia ixx="1e-6" ixy="0" ixz="0" iyy="1e-6" iyz="0" izz="1e-6" />
-		</inertial>
-	</link>
-	<!-- Drive controller -->
-	<gazebo>
-		<plugin name="skid_steer_drive_controller" filename="libgazebo_ros_skid_steer_drive.so">
-			<updateRate>100.0</updateRate>
-			<robotNamespace>/</robotNamespace>
-			<leftFrontJoint>base_to_wheel1</leftFrontJoint>
-			<rightFrontJoint>base_to_wheel3</rightFrontJoint>
-			<leftRearJoint>base_to_wheel2</leftRearJoint>
-			<rightRearJoint>base_to_wheel4</rightRearJoint>
-			<wheelSeparation>4</wheelSeparation>
-			<wheelDiameter>0.1</wheelDiameter>
-			<robotBaseFrame>base_link</robotBaseFrame>
-			<torque>1</torque>
-			<topicName>cmd_vel</topicName>
-			<broadcastTF>0</broadcastTF>
-		</plugin>
-	</gazebo>
 </robot>

File: ws_ros1/src/robot_description/urdf/robot1_base_01_cam_hok.xacro (robot description, xacro)
@@ -22,5 +22,5 @@
 		<xacro:default_inertial mass="0.0001"/>
 	</link>
-	<xacro:include filename="$(find robot1_description)/urdf/robot.gazebo" />
+	<xacro:include filename="$(find robot_description)/urdf/robot.gazebo" />
 	<gazebo reference="base_footprint">
 		<material>Gazebo/Green</material>
@@ -187,5 +187,5 @@
 			<origin xyz="0 0 0" rpy="0 0 0"/>
 			<geometry>
-				<mesh filename="package://robot1_description/meshes/hokuyo.dae"/>
+				<mesh filename="package://robot_description/meshes/hokuyo.dae"/>
 			</geometry>
 		</visual>

File: ws_ros1/src/robot_description/urdf/robot1_base_02.xacro (robot description, xacro)
@@ -6,5 +6,4 @@
 	<xacro:property name="length_wheel" value="0.05" />
 	<xacro:property name="radius_wheel" value="0.05" />
-	<xacro:property name="camera_link" value="0.05" />
 	<xacro:macro name="default_inertial" params="mass">
 		<inertial>
@@ -13,4 +12,5 @@
 		</inertial>
 	</xacro:macro>
+	<xacro:include filename="$(find robot_description)/urdf/robot.gazebo" />
 	<link name="base_footprint">
 		<visual>
@@ -22,5 +22,4 @@
 		<xacro:default_inertial mass="0.0001"/>
 	</link>
-	<xacro:include filename="$(find robot1_description)/urdf/robot.gazebo" />
 	<gazebo reference="base_footprint">
 		<material>Gazebo/Green</material>
@@ -38,6 +37,6 @@
 			</geometry>
 			<origin rpy="0 0 1.54" xyz="0 0 0.05"/>
-			<material name="white">
-				<color rgba="1 1 1 1"/>
+			<material name="darkblue">
+				<color rgba=".1 .1 .5 1"/>
 			</material>
 		</visual>
@@ -141,32 +140,3 @@
 		<origin rpy="1.5707 0 0" xyz="-0.1 -0.15 0"/>
 	</joint>
-	<joint name="camera_joint" type="fixed">
-		<axis xyz="0 1 0" />
-		<origin xyz="0.125 0 0.125" rpy="0 0 0"/>
-		<parent link="base_link"/>
-		<child link="camera_link"/>
-	</joint>
-	<!-- Camera -->
-	<link name="camera_link">
-		<collision>
-			<origin xyz="0 0 0" rpy="0 0 0"/>
-			<geometry>
-				<box size="0.05 0.05 0.05"/>
-			</geometry>
-		</collision>
-		<visual>
-			<origin xyz="0 0 0" rpy="0 0 0"/>
-			<geometry>
-				<box size="0.05 0.05 0.05"/>
-			</geometry>
-			<material name="red">
-				<color rgba="1 0 0 1"/>
-			</material>
-		</visual>
-		<inertial>
-			<mass value="1e-5" />
-			<origin xyz="0 0 0" rpy="0 0 0"/>
-			<inertia ixx="1e-6" ixy="0" ixz="0" iyy="1e-6" iyz="0" izz="1e-6" />
-		</inertial>
-	</link>
 </robot>

File: ws_ros1/src/robot_description/urdf/robot1_base_03.xacro (robot description, xacro)
@@ -6,4 +6,5 @@
 	<xacro:property name="length_wheel" value="0.05" />
 	<xacro:property name="radius_wheel" value="0.05" />
+	<xacro:property name="camera_link" value="0.05" />
 	<xacro:macro name="default_inertial" params="mass">
 		<inertial>
@@ -12,5 +13,4 @@
 		</inertial>
 	</xacro:macro>
-	<xacro:include filename="$(find robot1_description)/urdf/robot.gazebo" />
 	<link name="base_footprint">
 		<visual>
@@ -22,4 +22,5 @@
 		<xacro:default_inertial mass="0.0001"/>
 	</link>
+	<xacro:include filename="$(find robot_description)/urdf/robot.gazebo" />
 	<gazebo reference="base_footprint">
 		<material>Gazebo/Green</material>
@@ -37,6 +38,6 @@
 			</geometry>
 			<origin rpy="0 0 1.54" xyz="0 0 0.05"/>
-			<material name="darkblue">
-				<color rgba=".1 .1 .5 1"/>
+			<material name="white">
+				<color rgba="1 1 1 1"/>
 			</material>
 		</visual>
@@ -140,3 +141,58 @@
 		<origin rpy="1.5707 0 0" xyz="-0.1 -0.15 0"/>
 	</joint>
+	<joint name="camera_joint" type="fixed">
+		<axis xyz="0 1 0" />
+		<origin xyz="0.125 0 0.125" rpy="0 0 0"/>
+		<parent link="base_link"/>
+		<child link="camera_link"/>
+	</joint>
+	<!-- Camera -->
+	<link name="camera_link">
+		<collision>
+			<origin xyz="0 0 0" rpy="0 0 0"/>
+			<geometry>
+				<box size="0.05 0.05 0.05"/>
+			</geometry>
+		</collision>
+		<visual>
+			<origin xyz="0 0 0" rpy="0 0 0"/>
+			<geometry>
+				<box size="0.05 0.05 0.05"/>
+			</geometry>
+			<material name="red">
+				<color rgba="1 0 0 1"/>
+			</material>
+		</visual>
+		<inertial>
+			<mass value="1e-5" />
+			<origin xyz="0 0 0" rpy="0 0 0"/>
+			<inertia ixx="1e-6" ixy="0" ixz="0" iyy="1e-6" iyz="0" izz="1e-6" />
+		</inertial>
+	</link>
+	<joint name="hokuyo_joint" type="fixed">
+		<axis xyz="0 1 0" />
+		<origin xyz="0.125 0.05 0.125" rpy="0 0 0"/>
+		<parent link="base_link"/>
+		<child link="hokuyo_link"/>
+	</joint>
+	<!-- Hokuyo Laser -->
+	<link name="hokuyo_link">
+		<collision>
+			<origin xyz="0 0 0" rpy="0 0 0"/>
+			<geometry>
+				<box size="0.1 0.1 0.1"/>
+			</geometry>
+		</collision>
+		<visual>
+			<origin xyz="0 0 0" rpy="0 0 0"/>
+			<geometry>
+				<mesh filename="package://robot_description/meshes/hokuyo.dae"/>
+			</geometry>
+		</visual>
+		<inertial>
+			<mass value="1e-5" />
+			<origin xyz="0 0 0" rpy="0 0 0"/>
+			<inertia ixx="1e-6" ixy="0" ixz="0" iyy="1e-6" iyz="0" izz="1e-6" />
+		</inertial>
+	</link>
 </robot>

File: ws_ros1/src/robot_description/urdf/robot1_base_04.xacro (robot description, xacro)
@@ -22,5 +22,5 @@
 		<xacro:default_inertial mass="0.0001"/>
 	</link>
-	<xacro:include filename="$(find robot1_description)/urdf/robot.gazebo" />
+	<xacro:include filename="$(find robot_description)/urdf/robot.gazebo" />
 	<gazebo reference="base_footprint">
 		<material>Gazebo/Green</material>
@@ -118,5 +118,5 @@
 		<parent link="base_link"/>
 		<child link="wheel_1"/>
-		<origin rpy="1.5707 0 0" xyz="0.1 0.15 0"/>
+		<origin rpy="-1.5707 0 0" xyz="0.1 0.15 0"/>
 		<axis xyz="0 0 1" />
 	</joint>
@@ -127,5 +127,5 @@
 		<parent link="base_link"/>
 		<child link="wheel_2"/>
-		<origin rpy="1.5707 0 0" xyz="-0.1 0.15 0"/>
+		<origin rpy="-1.5707 0 0" xyz="-0.1 0.15 0"/>
 	</joint>
 	<joint name="base_to_wheel3" type="continuous">
@@ -133,5 +133,5 @@
 		<axis xyz="0 0 1" />
 		<child link="wheel_3"/>
-		<origin rpy="1.5707 0 0" xyz="0.1 -0.15 0"/>
+		<origin rpy="-1.5707 0 0" xyz="0.1 -0.15 0"/>
 	</joint>
 	<joint name="base_to_wheel4" type="continuous">
@@ -139,6 +139,7 @@
 		<axis xyz="0 0 1" />
 		<child link="wheel_4"/>
-		<origin rpy="1.5707 0 0" xyz="-0.1 -0.15 0"/>
-	</joint>
+		<origin rpy="-1.5707 0 0" xyz="-0.1 -0.15 0"/>
+	</joint>
+	<!-- Camera joint -->
 	<joint name="camera_joint" type="fixed">
 		<axis xyz="0 1 0" />
@@ -170,8 +171,9 @@
 		</inertial>
 	</link>
+	<!-- Hokuyo joint -->
 	<joint name="hokuyo_joint" type="fixed">
+		<origin xyz="0.125 0.05 0.125" rpy="0 0 0"/>
+		<parent link="base_link"/>
 		<axis xyz="0 1 0" />
-		<origin xyz="0.125 0.05 0.125" rpy="0 0 0"/>
-		<parent link="base_link"/>
 		<child link="hokuyo_link"/>
 	</joint>
@@ -187,5 +189,5 @@
 			<origin xyz="0 0 0" rpy="0 0 0"/>
 			<geometry>
-				<mesh filename="package://robot1_description/meshes/hokuyo.dae"/>
+				<mesh filename="package://robot_description/meshes/hokuyo.dae"/>
 			</geometry>
 		</visual>
@@ -196,3 +198,20 @@
 		</inertial>
 	</link>
+	<!-- Drive controller -->
+	<gazebo>
+		<plugin name="skid_steer_drive_controller" filename="libgazebo_ros_skid_steer_drive.so">
+			<updateRate>100.0</updateRate>
+			<robotNamespace>/</robotNamespace>
+			<leftFrontJoint>base_to_wheel1</leftFrontJoint>
+			<rightFrontJoint>base_to_wheel3</rightFrontJoint>
+			<leftRearJoint>base_to_wheel2</leftRearJoint>
+			<rightRearJoint>base_to_wheel4</rightRearJoint>
+			<wheelSeparation>4</wheelSeparation>
+			<wheelDiameter>0.1</wheelDiameter>
+			<robotBaseFrame>base_link</robotBaseFrame>
+			<torque>1</torque>
+			<topicName>cmd_vel</topicName>
+			<broadcastTF>0</broadcastTF>
+		</plugin>
+	</gazebo>
 </robot>

File: ws_ros1/src/robot_description/urdf/robot1_physics.urdf (robot description, URDF)
Before this commit: robot origins, 12 links, 11 joints
Links:
- link left_gripper: geometry collision box size=0.1 .1 .1; visual mesh filename=package://robot_description/meshes/gripper_v0/l_finger.dae
- link left_tip: geometry collision box size=0.1 .1 .1; visual mesh filename=package://robot_description/meshes/gripper_v0/l_finger_tip.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
- link right_gripper: geometry collision box size=0.1 .1 .1; visual mesh filename=package://robot_description/meshes/gripper_v0/l_finger.dae
- link right_tip: geometry collision box size=0.1 .1 .1; visual mesh filename=package://robot_description/meshes/gripper_v0/l_finger_tip.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

File: ws_ros1/src/robot_description/urdf/robot_car_dae.urdf (robot description, URDF)
Before this commit: robot robot1, 1 links, 0 joints
Links:
- link base_link: geometry visual mesh filename=package://robot_description/meshes/bot.dae scale=1 1 1
